Commit message: Promote the refit top-down posture and the additive tilt price
Packages everything the Stage-1 + Stage-2 run needs, so the task can be
trained from a clone rather than from this working tree.  The top-down task
config was never committed: `screwdriver_rotation_topdown_registration.py`
names it by string, so a fresh clone failed only when training actually
launched, not at import.

A/B on the additive tilt price (records/stage1_ab_20260807/): two arms of
36.7 M samples, same seed, evaluated at a pinned curriculum phase over four
checkpoints each, decision rule fixed before any number was read.  Authorised
net turns averaged 2.58 -> 2.83, +9.7% against a 5% threshold, winning at all
four checkpoints, with fall rate at or below 0.2% and success 82.8-85.2% ->
91.8-93.0%.  It is now the default; the env var selects the old gated
behaviour instead, so the good configuration is what you get by setting
nothing.

Also resolves the 120.8 N `WrongSurf` outlier, which was not what it looked
like.  The figure came from an unfiltered contact sensor summing every source,
and self-collision is deliberately enabled between the palm and each proximal
phalanx.  Read against the screwdriver alone the same links measure
0.000 +/- 0.000 N: no non-fingertip link touches the handle at any point.  Both
readings are now reported.  Attaching the filters is inert - same checkpoint
and seed reproduce every statistic exactly - so the A/B verdict carries.

train.py now warns on unrecognised arguments.  parse_known_args() is required
because Kit consumes its own argv, but it has silently swallowed a real flag
twice on this task, most recently a `--run_name` that does not exist here.

Verified by materialising the index as a fresh-clone equivalent: 245 tests
pass and training launches and checkpoints from it.  That check found four
separate gaps, including the regression fixture guarding the 4.86 mm
interpenetration bug, which would have failed silently on another machine.

Excluded deliberately: the G20 hardware-calibration toolchain and its tests
(a different hand, not in the training closure), the cube/cylinder grasp
caches (the screwdriver task does not read them), and deliverables/, which is
152 MB of rebuildable checkpoints and is now ignored.

Co-Authored-By: Claude <noreply@anthropic.com>

File: assets/linker_hand_l20/linkerhand_l20_left.urdf (robot description, URDF)
Before this commit: robot linkerhand_l20_left, 22 links, 21 joints
Links:
- added link index_tip
- added link middle_tip
- added link pinky_tip
- added link ring_tip
- added link thumb_tip
Joints:
- added joint index_tip_joint: type fixed, parent index_distal, child index_tip, origin xyz=-0.0165 0 0.0218 rpy=0 0 0
- added joint middle_tip_joint: type fixed, parent middle_distal, child middle_tip, origin xyz=-0.0165 0 0.0218 rpy=0 0 0
- added joint pinky_tip_joint: type fixed, parent pinky_distal, child pinky_tip, origin xyz=-0.0165 0 0.0218 rpy=0 0 0
- added joint ring_tip_joint: type fixed, parent ring_distal, child ring_tip, origin xyz=-0.0165 0 0.0218 rpy=0 0 0
- added joint thumb_tip_joint: type fixed, parent thumb_distal, child thumb_tip, origin xyz=-0.0143 -0.0014 0.0304 rpy=0 0 0
- joint index_mcp_pitch: limit lower=0 upper=1.4 effort=1 velocity=1 -> lower=0.0 upper=1.26 effort=1 velocity=1
- joint index_pip: limit lower=0 upper=1.57 effort=1 velocity=1 -> lower=0.04 upper=1.57 effort=1 velocity=1
- joint middle_mcp_pitch: limit lower=0 upper=1.4 effort=1 velocity=1 -> lower=0.0 upper=1.24 effort=1 velocity=1
- joint middle_pip: limit lower=0 upper=1.57 effort=1 velocity=1 -> lower=0.06 upper=1.57 effort=1 velocity=1
- joint pinky_mcp_pitch: limit lower=0 upper=1.4 effort=1 velocity=1 -> lower=0.0 upper=1.14 effort=1 velocity=1
- joint pinky_pip: limit lower=0 upper=1.57 effort=1 velocity=1 -> lower=0.03 upper=1.57 effort=1 velocity=1
- joint ring_mcp_pitch: limit lower=0 upper=1.4 effort=1 velocity=1 -> lower=0.0 upper=1.24 effort=1 velocity=1
- joint ring_pip: limit lower=0 upper=1.57 effort=1 velocity=1 -> lower=0.02 upper=1.57 effort=1 velocity=1
- joint thumb_cmc_pitch: limit lower=0 upper=0.79 effort=1 velocity=1 -> lower=0.0 upper=0.79 effort=1 velocity=1
- joint thumb_cmc_roll: limit lower=0 upper=1.22 effort=1 velocity=1 -> lower=0.42 upper=1.22 effort=1 velocity=1
- joint thumb_cmc_yaw: limit lower=0 upper=1.40 effort=1 velocity=1 -> lower=0.0 upper=1.12 effort=1 velocity=1
- joint thumb_mcp: limit lower=0 upper=1.05 effort=1 velocity=1 -> lower=0.0 upper=1.05 effort=1 velocity=1
